File: PGA-103+ LNA/PGA-103+ LNA.brd (EAGLE design)
At the start: 90.2 x 56.2 mm, 42 parts, among them IC1 7805DT, K1 351, K2 351, K3 351, K4 351, K5 351, K6 351, X1 SMA, X2 SMA

Commit message: First commit
Parts:
- moved C3 6.25 mm to (33.0, 38.1), turned to 90 degrees
- moved C1 0.63 mm to (28.6, 43.8), turned to 315 degrees
Routing:
- net VCC: track 238.3 -> 241.3 mm
- net N$14: track 5.00 -> 6.54 mm
- net N$16: track 34.3 -> 33.0 mm
- net N$17: track 33.7 -> 32.4 mm
- net GND: vias 231 -> 279
