File: PGA-103+ LNA Mod2/PGA-103+ LNA Mod2.brd (EAGLE design)
At the start: 97.8 x 53 mm, 42 parts, among them IC1 7805DT, K1 G2RE, K2 G2RE, K3 G2RE, K4 G2RE, X1 SMA, X2 SMA

Commit message: First commit
Parts:
- added C15, C16: 1n, rcl:C1206
Connections:
- net GND: now also C15.2, C16.2
- net VCC: now also C15.1, C16.1
Routing:
- net GND: track 40.2 -> 70.9 mm, vias 384 -> 386
- net RF_BYPASS: track 132.6 -> 141.4 mm, vias 0 -> 6
- net ANT: track 31.9 -> 37.9 mm, vias 0 -> 3
- net TRX: track 32.5 -> 35.9 mm, vias 0 -> 3
