File: Relay Sequencer/Relay Sequencer.sch (EAGLE design)
At the start: 22 parts, among them IC1 MEGA16-A, IC2 ULN2003AD

Commit message: First commit
Parts:
- removed JP3: (no value), pinhead:PINHD-1X2
- added C10, C13, C14, C15, C7, C8, C9: (no value), rcl:C-EUC1206
- added C11: (no value), rcl:CPOL-EUE5-8.5
- added C12: (no value), rcl:CPOL-EUE5-13
- added D2: 1N400x, diode:1N4148DO35-10
- added H1, H2, H3, H4: MOUNT-PAD, holes:MOUNT-PAD-SQUARE2.8
- added IC3: 7805DT, linear:7805DT
- added IC4: 74HC244DW, 74xx-eu:74HC244DW
- added J1, J2, J3, J4, J5, J6: (no value), con-amp:MTA02-156
- added K1, K2, K3, K4: 351, relay:351
- added LED5, LED6: (no value), led:LED3MM
- added R6, R7: (no value), rcl:R-US_M1206
- JP1: device pinhead:PINHD-2X4 -> pinhead:PINHD-2X5
- JP2: device pinhead:PINHD-2X5 -> pinhead:PINHD-2X4
Connections:
- removed net !SIG: D1.A, IC1.(INT1)PD3
- new net BE_1: IC4A.Y1, JP2.1
- new net BE_2: IC4A.Y2, JP2.3
- new net BE_3: IC4A.Y3, JP2.5
- new net BE_4: IC4A.Y4, JP2.7
- new net N$10: LED6.A, R7.1
- new net N$7: LED5.A, R6.1
- new net N$8: C4.1, D1.C, J1.2
- new net N$9: D2.A, J2.1
- new net R1A: J3.1, K12.P, K13.P
- new net R1B: J3.2, K12.S, K13.S
- new net R2A: J4.1, K22.P, K23.P
- new net R2B: J4.2, K22.S, K23.S
- new net R3A: J5.1, K32.P, K33.P
- new net R3B: J5.2, K32.S, K33.S
- new net R4A: J6.1, K42.P, K43.P
- new net R4B: J6.2, K42.S, K43.S
- net !PTT: now also C7.1, D1.A, IC1.(INT1)PD3; no longer D1.C
- net !RST: now also C8.1, JP1.5; no longer C3.1, JP2.5
- net +12V: now also C10.1, C11.+, C12.+, C13.1, C9.1, D2.C, IC3.VI, K11.1, K21.1, K31.1, K41.1
- net +5V: now also C14.1, C15.1, C2.1, C3.1, IC3.VO, IC4P.VCC, JP1.2, R7.2; no longer C4.1, C5.1, JP2.2
- net EN_1: now also IC1.(ADC4)PA4, IC4A.A1, R2.2; no longer IC1.(ADC7)PA7, JP1.1, R4.2
- net EN_2: now also IC1.(ADC5)PA5, IC4A.A2, R3.2; no longer IC1.(ADC6)PA6, JP1.3, R5.2
- net EN_3: now also IC1.(ADC6)PA6, IC4A.A3, R4.2; no longer IC1.(ADC5)PA5, JP1.5, R2.2
- net EN_4: now also IC1.(ADC7)PA7, IC4A.A4, R5.2; no longer IC1.(ADC4)PA4, JP1.7, R3.2
- net EVENT_1: now also K11.2
- net EVENT_2: now also K21.2
- net EVENT_3: now also K31.2
- net EVENT_4: now also K41.2
- net GND: now also C10.2, C11.-, C12.-, C13.2, C14.2, C15.2, C7.2, C8.2, C9.2, IC3.GND, IC4A.G, IC4B.A1, IC4B.A2, IC4B.A3, IC4B.A4, IC4B.G, IC4P.GND, J1.1, J2.2, JP1.10, JP2.2, JP2.4, JP2.6, LED5.C, LED6.C; no longer JP1.2, JP1.4, JP1.6, JP2.10, JP3.2
- net MISO: now also JP1.9; no longer JP2.9
- net MOSI: now also JP1.1; no longer JP2.1
- net N$1: now also C5.1; no longer C1.1
- net N$2: now also C1.1; no longer C2.1
- net PTT_OK: now also R6.2; no longer JP3.1
- net SCK: now also JP1.7; no longer JP2.7
Other:
- moved on the sheet: C1, C2, C3, C4, C5, C6, D1, IC1, IC2, LED1, LED2, LED3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
