File: Relay Sequencer/Relay Sequencer.brd (EAGLE design)
At the start: 95.2 x 81.3 mm, 51 parts, among them IC1 MEGA16-A, IC2 ULN2003AD, IC3 7805DT, IC4 74HC244DW, K1 351, K2 351, K3 351, K4 351

Commit message: First commit
Routing:
- net +12V: track 299.3 -> 338.5 mm
- net GND: track 367.3 -> 346.3 mm
- net R2A: track 40.6 -> 32.5 mm
- net N$8: track 86.8 -> 88.1 mm
